Commit message: Converted macros format to SDF (was URDF)

File: simulation/models/cones/cone.sdf.xacro (robot description, xacro)
@@ -1,4 +1,4 @@
 <?xml version="1.0"?>
-<robot xmlns:xacro="http://ros.org/wiki/xacro">
+<sdf version='1.7' xmlns:xacro="http://ros.org/wiki/xacro">
     <!-- Macro to define a cone -->
     <xacro:macro name="cone" params="name type pose">
@@ -74,3 +74,3 @@
     </model>
     </xacro:macro>
-</robot>
+</sdf>

File: simulation/models/vehicle/ads_dv.xacro (robot description, xacro)
@@ -1,106 +1,106 @@
 <?xml version="1.0" ?>
-<robot xmlns:xacro="http://www.ros.org/wiki/xacro" name="ads_dv">
-    <!-- Wheels and Joints -->
-    <xacro:include filename="$(find simulation)/models/vehicle/wheels.xacro" />
-    <link name='chassis'>
-        <inertial>
-            <mass value="278"/>
-            <inertia ixx="14.38" ixy="0" ixz="0" iyy="178.90" iyz="0" izz="175.68"/>
-        </inertial>
-        <visual name='visual'>
-            <origin xyz="0 0 0"/>
-            <geometry>
-                <mesh filename="package://simulation/models/vehicle/ads-dv.stl" scale="1 1 1"/>
-            </geometry>
-            <material name="chassis_mat">
-                <color rgba="0.0 0.2 0.13 1"/>
-            </material>
-        </visual>
-        <collision name='collision'>
-            <geometry>
-                <box size="2.7 0.489 0.414"/>
-            </geometry>
-        </collision>
-    </link>
-    <!-- Base Link -->
-    <link name='base_link'>
-        <visual name="visual">
-            <geometry>
-                <box size="0.01 0.01 0.01"/>
-            </geometry>
-        </visual>
-        <inertial> <!-- Needed to disable lumping -->
-            <mass value="0.001"/>
-            <inertia ixx="0.001" ixy="0" ixz="0" iyy="0.001" iyz="0" izz="0.001"/>
-        </inertial>
-    </link>
-    <!-- Steering Links and Joints-->
-    <link name="front_left_wheel_steering_link">
-        <inertial>
-            <mass value="0.001"/>
-            <inertia ixx="0.001" ixy="0" ixz="0" iyy="0.001" iyz="0" izz="0.001"/>
-        </inertial>
-        <visual name="steering_link_visual">
-            <geometry>
-                <cylinder length="0.1" radius="0.03"/>
-            </geometry>
-        </visual>
-    </link>
-    <joint name="front_left_wheel_steering_joint" type="revolute">
-        <parent link="chassis"/>
-        <child link="front_left_wheel_steering_link"/>
-        <axis xyz="0 0 1"/>
-        <limit lower="-0.424250477138" upper="0.424250477138" velocity="10000" effort="10000"/>
-        <origin xyz="0.767 0.47175 -0.0235" rpy="0 0 0"/>
-    </joint>
-    <link name="front_right_wheel_steering_link">
-        <inertial>
-            <mass value="0.001"/>
-            <inertia ixx="0.001" ixy="0" ixz="0" iyy="0.001" iyz="0" izz="0.001"/>
-        </inertial>
-        <visual name="steering_link_visual">
-            <geometry>
-                <cylinder length="0.1" radius="0.03"/>
-            </geometry>
-        </visual>
-    </link>
-    <joint name="front_right_wheel_steering_joint" type="revolute">
-        <parent link="chassis"/>
-        <child link="front_right_wheel_steering_link"/>
-        <axis xyz="0 0 1"/>
-        <limit lower="-0.424250477138" upper="0.424250477138" velocity="10000" effort="10000"/>
-        <origin xyz="0.767 -0.47175 -0.0235" rpy="0 0 0"/>
-    </joint>
-    <!-- Fixed Joints -->
-    <joint name="base_to_camera" type="fixed">
-        <parent link="base_link"/>
-        <child link="camera_link"/>
-        <origin xyz="0.4865 0 0.671" rpy="0 0 0"/>
-    </joint>
-    <gazebo reference='base_to_camera'>
-        <preserveFixedJoint>True</preserveFixedJoint>
-    </gazebo>
-    <joint name="base_to_velodyne" type="fixed">
-        <parent link="base_link"/>
-        <child link="velodyne"/>
-        <origin xyz="0.52 0 0.59946" rpy="0 0 0"/>
-    </joint>
-    <gazebo reference='base_to_velodyne'>
-        <preserveFixedJoint>True</preserveFixedJoint>
-    </gazebo>
-    <joint name="base_to_chassis" type="fixed">
-        <parent link="base_link"/>
-        <child link="chassis"/>
-        <origin xyz="0 0 0.307" rpy="0 0 0"/>
-    </joint>
-    <gazebo reference='base_to_chassis'>
-        <preserveFixedJoint>True</preserveFixedJoint>
-    </gazebo>
-    <!-- Sim (Stereo + Depth + Logical) Camera -->
-    <xacro:include filename="$(find simulation)/models/vehicle/sim_camera.xacro" />
-    <!-- Velodyne -->
-    <xacro:include filename="$(find simulation)/models/vehicle/velodyne.xacro" />
-    <!-- Ackermann Steering Plugin -->
-    <gazebo>
+<sdf version='1.11' xmlns:xacro="http://www.ros.org/wiki/xacro">
+    <model name='ads_dv' canonical_link='base_link'>
+        <!-- Base Link -->
+        <link name='base_link'>
+            <inertial>
+                <!-- Needed to disable lumping -->
+                <mass>0.001</mass>
+                <inertia>
+                    <ixx>0.001</ixx>
+                    <ixy>0</ixy>
+                    <ixz>0</ixz>
+                    <iyy>0.001</iyy>
+                    <iyz>0</iyz>
+                    <izz>0.001</izz>
+                </inertia>
+            </inertial>
+            <visual name='base_link_visual'>
+                <geometry>
+                    <box>
+                        <size>0.01 0.01 0.01</size>
+                    </box>
+                </geometry>
+            </visual>
+        </link>
+        <!-- Chassis -->
+        <link name='chassis'>
+            <pose relative_to='base_to_chassis'>0 0 0 0 0 0</pose>
+            <inertial>
+                <pose>0 0 0 0 0 0</pose>
+                <mass>278</mass>
+                <inertia>
+                    <ixx>14.38</ixx>
+                    <ixy>0</ixy>
+                    <ixz>0</ixz>
+                    <iyy>178.90</iyy>
+                    <iyz>0</iyz>
+                    <izz>175.68</izz>
+                </inertia>
+            </inertial>
+            <collision name='chassis_collision'>
+                <pose>0 0 0 0 0 0</pose>
+                <geometry>
+                    <box>
+                        <size>2.7 0.489 0.414</size>
+                    </box>
+                </geometry>
+            </collision>
+            <visual name='chassis_visual'>
+                <pose>0 0 0 0 0 0</pose>
+                <geometry>
+                    <mesh>
+                        <uri>model://simulation/models/vehicle/ads-dv.stl</uri>
+                        <scale>1 1 1</scale>
+                    </mesh>
+                </geometry>
+                <material>
+                    <diffuse>0 0.25 0.1625 1</diffuse>
+                    <ambient>0 0.25 0.1625 1</ambient>
+                </material>
+            </visual>
+            <sensor name='imu_sensor' type='imu'>
+                <always_on>1</always_on>
+                <update_rate>300</update_rate>
+                <visualize>true</visualize>
+                <topic>imu</topic>
+            </sensor>
+        </link>
+         <!-- Wheels and Joints -->
+        <xacro:include filename="$(find simulation)/models/vehicle/wheel.xacro" />
+        <xacro:wheel name="front_left_wheel" parent="front_left_wheel_steering_link" x="0" y="0.09825" z="0" roll="-1.5707" pitch="0" yaw="0"/>
+        <xacro:wheel name="front_right_wheel" parent="front_right_wheel_steering_link" x="0" y="-0.09825" z="0" roll="-1.5707" pitch="0" yaw="0"/>
+        <xacro:wheel name="rear_left_wheel" parent="chassis" x="-0.767" y="0.57" z="-0.0235" roll="-1.5707" pitch="0" yaw="0"/>
+        <xacro:wheel name="rear_right_wheel" parent="chassis" x="-0.767" y="-0.57" z="-0.0235" roll="-1.5707" pitch="0" yaw="0"/>
+        <!-- Steering Links and Joints -->
+        <xacro:include filename="$(find simulation)/models/vehicle/steering.xacro" />
+        <xacro:steering name="front_left_wheel_steering" parent="chassis" limit="0.424250477138" x="0.767" y="0.47175" z="-0.0235" roll="0" pitch="0" yaw="0"/>
+        <xacro:steering name="front_right_wheel_steering" parent="chassis" limit="0.424250477138" x="0.767" y="-0.47175" z="-0.0235" roll="0" pitch="0" yaw="0"/>
+        <!-- Fixed Joints -->
+        <joint name='base_to_camera' type='fixed'>
+            <pose relative_to='base_link'>0.4865 0 0.671 0 0 0</pose>
+            <parent>base_link</parent>
+            <child>camera_link</child>
+        </joint>
+        <joint name='base_to_logical_camera' type='fixed'>
+            <pose relative_to='base_link'>0.4865 0 0.671 0 0 0</pose>
+            <parent>base_link</parent>
+            <child>logical_camera_link</child>
+        </joint>
+        <joint name='base_to_velodyne' type='fixed'>
+            <pose relative_to='base_link'>0.52 0 0.59946 0 0 0</pose>
+            <parent>base_link</parent>
+            <child>velodyne</child>
+        </joint>
+        <joint name='base_to_chassis' type='fixed'>
+            <pose relative_to='base_link'>0 0 0.307 0 0 0</pose>
+            <parent>base_link</parent>
+            <child>chassis</child>
+        </joint>
+        <!-- Sim (Stereo + Depth + Logical) Camera -->
+        <xacro:include filename="$(find simulation)/models/vehicle/sim_camera.xacro" />
+        <!-- Velodyne -->
+        <xacro:include filename="$(find simulation)/models/vehicle/velodyne.xacro" />
+        <!-- Ackermann Steering Plugin -->
         <plugin filename="gz-sim-ackermann-steering-system" name="gz::sim::systems::AckermannSteering">
             <left_joint>front_left_wheel_joint</left_joint>
@@ -121,5 +121,5 @@
             <min_acceleration>-5.2</min_acceleration>
             <max_acceleration>5.2</max_acceleration>
-            <frame_id>ads_dv</frame_id>
+            <frame_id>odom</frame_id>
             <child_frame_id>base_link</child_frame_id>
         </plugin>
@@ -127,7 +127,10 @@
             <render_engine>ogre2</render_engine>
         </plugin>
-         <plugin name="gz::sim::systems::JointStatePublisher" filename="gz-sim-joint-state-publisher-system">
+            <plugin name="gz::sim::systems::JointStatePublisher" filename="gz-sim-joint-state-publisher-system">
             <topic>/model/ads_dv/joint_state</topic>
         </plugin>
-    </gazebo>
-</robot>
+        <plugin filename="gz-sim-imu-system"
+            name="gz::sim::systems::Imu">
+        </plugin>
+    </model>
+</sdf>

File: simulation/models/vehicle/sim_camera.xacro (robot description, xacro)
@@ -1,24 +1,40 @@
 <?xml version="1.0" ?>
-<robot xmlns:xacro="http://www.ros.org/wiki/xacro" name="ZED-2i">
+<sdf version='1.7' xmlns:xacro="http://www.ros.org/wiki/xacro" name="ZED-2i">
     <!-- Depth Camera -->
-    <link name="camera_link">
-        <visual name="visual">
+    <link name='camera_link'>
+        <pose relative_to='base_to_camera'>0 0 0 0 0 0</pose>
+        <inertial>
+            <mass>0.001</mass>
+            <inertia>
+                <ixx>0.001</ixx>
+                <ixy>0</ixy>
+                <ixz>0</ixz>
+                <iyy>0.001</iyy>
+                <iyz>0</iyz>
+                <izz>0.001</izz>
+            </inertia>
+        </inertial>
+        <visual name='camera_link_visual'>
             <geometry>
-                <box size="0.0431 0.17525 0.03025"/>
+                <box>
+                    <size>0.0431 0.17525 0.03025</size>
+                </box>
             </geometry>
         </visual>
+    </link>
+    <link name='camera_link_optical'>
+        <pose relative_to='camera_to_optical'>0 0 0 0 0 0</pose>
         <inertial>
-            <mass value="0.001"/>
-            <inertia ixx="0.001" ixy="0" ixz="0" iyy="0.001" iyz="0" izz="0.001"/>
+            <mass>0.001</mass>
+            <inertia>
+                <ixx>0.001</ixx>
+                <ixy>0</ixy>
+                <ixz>0</ixz>
+                <iyy>0.001</iyy>
+                <iyz>0</iyz>
+                <izz>0.001</izz>
+            </inertia>
         </inertial>
-    </link>
-    <link name="camera_link_optical">
-        <inertial>
-            <mass value="0.001"/>
-            <inertia ixx="0.001" ixy="0" ixz="0" iyy="0.001" iyz="0" izz="0.001"/>
-        </inertial>
-    </link>
-    <gazebo reference="camera_link_optical">
-        <sensor name="zed2i_depth_camera" type="rgbd_camera">
+        <sensor name='zed2i_depth_camera' type='rgbd_camera'>
             <gz_frame_id>camera_link_optical</gz_frame_id>
             <update_rate>30</update_rate>
@@ -26,5 +42,5 @@
             <camera>
                 <camera_info_topic>camera_info</camera_info_topic>
-                <horizontal_fov>1.9198622</horizontal_fov> <!-- 110 degrees -->
+                <horizontal_fov>1.22173</horizontal_fov>
                 <image>
                     <width>640</width>
@@ -37,7 +53,10 @@
                 </clip>
                 <noise>
+                    <!-- This is an unrealistic depth noise model, but that's what's available currently -->
+                    <!-- Probably a good idea to simulate a stereo camera and use a ROS node to estimate depth -->
+                    <!-- Or ditch Gazebo altogether -->
                     <type>gaussian</type>
                     <mean>0.0</mean>
-                    <stddev>0.007</stddev> <!-- idk where this comes from-->
+                    <stddev>0.007</stddev>
                 </noise>
                 <distortion>
@@ -50,22 +69,26 @@
             </camera>
         </sensor>
-    </gazebo>
-    <joint name="camera_to_optical" type="fixed">
-        <parent link="camera_link"/>
-        <child link="camera_link_optical"/>
-        <origin xyz="0 0 0" rpy="0 0 0"/>
+    </link>
+    <joint name='camera_to_optical' type='fixed'>
+        <pose relative_to='camera_link'>0 0 0 0 0 0</pose>
+        <parent>camera_link</parent>
+        <child>camera_link_optical</child>
     </joint>
-    <gazebo reference='camera_to_optical'>
-        <preserveFixedJoint>True</preserveFixedJoint>
-    </gazebo>
     <!-- Logical Camera -->
     <link name='logical_camera_link'>
+        <pose relative_to='base_to_logical_camera'>0 0 0 0 0 0</pose>
         <inertial>
-            <mass value="0.001"/>
-            <inertia ixx="0.001" ixy="0" ixz="0" iyy="0.001" iyz="0" izz="0.001"/>
+            <mass>0.001</mass>
+            <inertia>
+                <ixx>0.001</ixx>
+                <ixy>0</ixy>
+                <ixz>0</ixz>
+                <iyy>0.001</iyy>
+                <iyz>0</iyz>
+                <izz>0.001</izz>
+            </inertia>
         </inertial>
-    </link>
-    <gazebo reference='logical_camera_link'>
         <sensor name='logical_camera' type='logical_camera'>
+            <gz_frame_id>camera_link_optical</gz_frame_id>
             <update_rate>30</update_rate>
             <topic>logical_camera</topic>
@@ -74,37 +97,10 @@
             <enable_metrics>true</enable_metrics>
             <logical_camera>
-            <near>1.5</near>
-            <far>35</far>
-            <aspect_ratio>1.333333333333333</aspect_ratio>
-            <horizontal_fov>1.9198622000000001</horizontal_fov>
+                <near>1.5</near>
+                <far>35</far>
+                <aspect_ratio>1.333333333333333</aspect_ratio>
+                <horizontal_fov>1.22173</horizontal_fov>
             </logical_camera>
         </sensor>
-    </gazebo>
-    <joint name='base_to_logical_camera' type='fixed'>
-        <parent link="base_link"/>
-        <child link="logical_camera_link"/>
-        <origin xyz="0.48649999999999999 0 0.67100000000000004" rpy="0 0 0"/>
-        <axis>
-            <dynamics>
-                <spring_reference>0</spring_reference>
-                <spring_stiffness>0</spring_stiffness>
-            </dynamics>
-            <xyz>0 0 1</xyz>
-            <limit>
-                <lower>-inf</lower>
-                <upper>inf</upper>
-            </limit>
-        </axis>
-        <physics>
-            <ode>
-                <limit>
-                <cfm>0</cfm>
-                <erp>0.20000000000000001</erp>
-                </limit>
-            </ode>
-        </physics>
-    </joint>
-    <gazebo reference='base_to_logical_camera'>
-        <preserveFixedJoint>True</preserveFixedJoint>
-    </gazebo>
-</robot>
+    </link>
+</sdf>
